File: Mimisbrunnr_PCB/controller.kicad_sch (KiCad schematic)
At the start: 12 parts, among them J1 Conn_01x04_Female, SW1 SW_Push, SW2 SW_Push, SW3 SW_Push, U1 ESP32-WROOM-32

Commit message: finalize schematic
Parts:
- added J10: Conn_01x06_Female, Connector_PinHeader_2.54mm:PinHeader_1x06_P2.54mm_Vertical, symbol Connector:Conn_01x06_Female
- added U3, U4, U5, U6, U7: MAX31856, Package_SO:TSSOP-14_4.4x5mm_P0.65mm, symbol Sensor_Temperature:MAX31856
Connections:
- net LED1: now also U1.9 (IO33); no longer U1.8 (IO32)
- net button+: now also U1.11 (IO26); no longer U1.31 (IO19)
- net button-: now also U1.10 (IO25); no longer U1.30 (IO18)
- net thc1_cs: now reaches U1.26 (IO4)
- net thc1_cs: now also U3.9 (~{CS})
- net thc2_cs: now reaches U1.27 (IO16)
- net thc2_cs: now also U4.9 (~{CS})
- net thc3_cs: now reaches U1.28 (IO17)
- net thc3_cs: now also U5.9 (~{CS})
- net mosi: now reaches U1.37 (IO23)
- net mosi: now also J10.2 (Pin_2), U3.12 (SDI), U4.12 (SDI), U5.12 (SDI), U6.12 (SDI), U7.12 (SDI)
- net Tank_thc_1: no longer names the net of U1.4 (SENSOR_VP)
- net Tank_thc_2: no longer names the net of U1.5 (SENSOR_VN)
- net Tank_thc_3: no longer names the net of U1.6 (I34)
- net Tank_thc_4: no longer names the net of U1.7 (I35)
- net Water_thc_1 renamed thc4_cs
- net thc4_cs: now also U6.9 (~{CS})
- new net +3.3V: J10.1 (Pin_1), U3.5 (AVDD), U3.8 (DVDD), U4.5 (AVDD), U4.8 (DVDD), U5.5 (AVDD), U5.8 (DVDD), U6.5 (AVDD), U6.8 (DVDD), U7.5 (AVDD), U7.8 (DVDD)
- new net Earth: J10.6 (Pin_6), U3.1 (AGND), U3.14 (DGND), U3.2 (BIAS), U4.1 (AGND), U4.14 (DGND), U4.2 (BIAS), U5.1 (AGND), U5.14 (DGND), U5.2 (BIAS), U6.1 (AGND), U6.14 (DGND), U6.2 (BIAS), U7.1 (AGND), U7.14 (DGND), U7.2 (BIAS)
- new net ext_cs: J10.5 (Pin_5)
- new net miso: J10.3 (Pin_3), U1.31 (IO19), U3.11 (SDO), U4.11 (SDO), U5.11 (SDO), U6.11 (SDO), U7.11 (SDO)
- new net sck: J10.4 (Pin_4), U1.30 (IO18), U3.10 (SCK), U4.10 (SCK), U5.10 (SCK), U6.10 (SCK), U7.10 (SCK)
- new net tank_thc_1+: U3.4 (T+)
- new net tank_thc_1-: U3.3 (T-)
- new net tank_thc_2+: U4.4 (T+)
- new net tank_thc_2-: U4.3 (T-)
- new net tank_thc_3+: U5.4 (T+)
- new net tank_thc_3-: U5.3 (T-)
- new net tank_thc_4+: U6.4 (T+)
- new net tank_thc_4-: U6.3 (T-)
- new net thc_water_cs: U1.8 (IO32), U7.9 (~{CS})
- new net water_thc+: U7.4 (T+)
- new net water_thc-: U7.3 (T-)
- no-connect marks 8 -> 18

Commit message: routing finished
Parts:
- removed J10: Conn_01x06_Female, Connector_PinHeader_2.54mm:PinHeader_1x06_P2.54mm_Vertical, symbol Connector:Conn_01x06_Female
- added C3, C4, C5, C6, C7, C8: C_Small, Capacitor_SMD:C_0805_2012Metric, symbol Device:C_Small
- added J10: Conn_01x04_Female, Connector_PinHeader_2.54mm:PinHeader_1x04_P2.54mm_Vertical, symbol Connector:Conn_01x04_Female
- added R10, R11: 4k7, Resistor_SMD:R_0805_2012Metric, symbol Device:R_Small
- renumbered U6 to U4, U4 to U5, U5 to U6
Connections:
- net +3V3 is gone; now on net +3.3V: D2.2 (A), J1.1 (Pin_1), R1.1, SW2.2, SW3.2, U1.2 (VDD)
- net Earth is gone; now on net GND: U3.1 (AGND), U3.14 (DGND), U3.2 (BIAS), U4.1 (AGND), U4.14 (DGND), U4.2 (BIAS), U5.1 (AGND), U5.14 (DGND), U5.2 (BIAS), U6.1 (AGND), U6.14 (DGND), U6.2 (BIAS), U7.1 (AGND), U7.14 (DGND), U7.2 (BIAS)
- net +3.3V: now also C3.1, C4.1, C5.1, C6.1, C7.1, C8.1, J10.1 (Pin_1), R10.1, R11.1
- net ESP32_RX: now also J10.3 (Pin_3)
- net ESP32_TX: now also J10.2 (Pin_2)
- net GND: now also C3.2, C4.2, C5.2, C6.2, C7.2, C8.2, J10.4 (Pin_4)
- net SCL: now also J1.2 (Pin_2), U1.37 (IO23), R11.2; no longer J1.3 (Pin_3)
- net SDA: now also J1.3 (Pin_3), U1.36 (IO22), R10.2; no longer J1.2 (Pin_2)
- net mosi: now also U1.33 (IO21); no longer U1.37 (IO23)
- net thc1_cs: now also U1.29 (IO5); no longer U1.26 (IO4)
- net thc2_cs: now also U1.28 (IO17); no longer U1.27 (IO16)
- net thc3_cs: now also U1.27 (IO16); no longer U1.28 (IO17)
- net thc4_cs: now also U1.26 (IO4); no longer U1.29 (IO5)
- net thc_water_cs: now also U1.24 (IO2); no longer U1.8 (IO32)
- net Relay2_CTRL: now reaches U1.23 (IO15)
- net Relay1 renamed Relay1_CTRL
- net Relay2: no longer names the net of U1.13 (IO14)
Other:
- moved on the sheet: J1

Commit message: Improve style
Parts:
- removed C3, C4, C5, C6, C7: C_Small, Capacitor_SMD:C_0805_2012Metric, symbol Device:C_Small
- removed U3, U4, U5, U6, U7: MAX31856, Package_SO:TSSOP-14_4.4x5mm_P0.65mm, symbol Sensor_Temperature:MAX31856
- J1, J10: value Conn_01x04_Female -> header_01x04
Connections:
- net miso renamed MISO
- net mosi renamed MOSI
- net sck renamed SCK
- no-connect marks 18 -> 8
Other:
- moved on the sheet: D1, R10, R11, R2
