File: Mimisbrunnr_PCB/power_circuit.kicad_sch (KiCad schematic)
At the start: 4 parts, among them J2 Conn_01x02_Female, U2 TLV76733DRVx

Commit message: finalize schematic
Parts:
- removed J2: Conn_01x02_Female, Connector_PinHeader_2.54mm:PinHeader_1x02_P2.54mm_Horizontal, symbol Connector:Conn_01x02_Female
- added J2: Jack-DC, Connector_AMASS:AMASS_XT30PW-M_1x02_P2.50mm_Horizontal, symbol Connector:Jack-DC
Connections:
- net +12V: now also J2.2
- net GND: now also J2.1
Other:
- note added: "Inverted because this and XT30 actually"
Changed lines of the file:
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@@
   (junction (at 149.352 86.614) (diameter 0) (color 0 0 0 0)
   )
-  (wire (pts (xy 117.856 89.408) (xy 117.856 91.694))
+  (wire (pts (xy 108.966 91.44) (xy 108.966 93.726))
     (stroke (width 0) (type default) (color 0 0 0 0))
   )
@@
     (stroke (width 0) (type default) (color 0 0 0 0))
   )
-  (wire (pts (xy 117.856 86.868) (xy 117.856 85.852))
+  (wire (pts (xy 108.966 86.36) (xy 108.966 85.344))
     (stroke (width 0) (type default) (color 0 0 0 0))
   )
-  (wire (pts (xy 117.856 86.868) (xy 114.3 86.868))
+  (wire (pts (xy 108.966 86.36) (xy 105.41 86.36))
     (stroke (width 0) (type default) (color 0 0 0 0))
   )
-  (wire (pts (xy 114.3 89.408) (xy 117.856 89.408))
+  (wire (pts (xy 105.41 91.44) (xy 108.966 91.44))
     (stroke (width 0) (type default) (color 0 0 0 0))
   )
@@
   (text "Linear Regulator" (at 149.352 76.454 0)
     (effects (font (size 2.5 2.5) (thickness 0.5) bold) (justify left bottom))
+  )
+  (text "Inverted because this and XT30 actually" (at 83.82 102.87 0)
+    (effects (font (size 1.27 1.27)) (justify left bottom))
+  )
+  (symbol (lib_id "Connector:Jack-DC") (at 97.79 88.9 0) (mirror x) (unit 1)
+    (in_bom yes) (on_board yes) (fields_autoplaced)
+    (property "Reference" "J2" (id 0) (at 91.44 87.6299 0)
+      (effects (font (size 1.27 1.27)) (justify right))
+    )
+    (property "Value" "Jack-DC" (id 1) (at 91.44 90.1699 0)
+      (effects (font (size 1.27 1.27)) (justify right))
+    )
+    (property "Footprint" "Connector_AMASS:AMASS_XT30PW-M_1x02_P2.50mm_Horizontal" (id 2) (at 99.06 87.884 0)
+      (effects (font (size 1.27 1.27)) hide)
+    )
+    (property "Datasheet" "~" (id 3) (at 99.06 87.884 0)
+      (effects (font (size 1.27 1.27)) hide)
+    )
+    (pin "1")
+    (pin "2")
   )
   (symbol (lib_id "Device:C") (at 149.352 90.424 0) (unit 1)
@@
     (pin "1")
   )
-  (symbol (lib_id "Connector:Conn_01x02_Female") (at 109.22 86.868 0) (mirror y) (unit 1)
+  (symbol (lib_id "power:+12V") (at 108.966 85.344 0) (mirror y) (unit 1)
     (in_bom yes) (on_board yes) (fields_autoplaced)
-    (property "Reference" "J2" (id 0) (at 108.5088 87.3033 0)
-      (effects (font (size 1.27 1.27)) (justify left))
-    )
-    (property "Value" "Conn_01x02_Female" (id 1) (at 108.5088 89.8402 0)
-      (effects (font (size 1.27 1.27)) (justify left))
-    )
-    (property "Footprint" "Connector_PinHeader_2.54mm:PinHeader_1x02_P2.54mm_Horizontal" (id 2) (at 109.22 86.868 0)
+    (property "Reference" "#PWR013" (id 0) (at 108.966 89.154 0)
       (effects (font (size 1.27 1.27)) hide)
     )
-    (property "Datasheet" "~" (id 3) (at 109.22 86.868 0)
+    (property "Value" "+12V" (id 1) (at 108.966 81.7682 0))
+    (property "Footprint" "" (id 2) (at 108.966 85.344 0)
       (effects (font (size 1.27 1.27)) hide)
     )
-    (pin "1")
-    (pin "2")
-  )
-  (symbol (lib_id "power:+12V") (at 117.856 85.852 0) (mirror y) (unit 1)
-    (in_bom yes) (on_board yes) (fields_autoplaced)
-    (property "Reference" "#PWR013" (id 0) (at 117.856 89.662 0)
-      (effects (font (size 1.27 1.27)) hide)
-    )
-    (property "Value" "+12V" (id 1) (at 117.856 82.2762 0))
-    (property "Footprint" "" (id 2) (at 117.856 85.852 0)
-      (effects (font (size 1.27 1.27)) hide)
-    )
-    (property "Datasheet" "" (id 3) (at 117.856 85.852 0)
+    (property "Datasheet" "" (id 3) (at 108.966 85.344 0)
       (effects (font (size 1.27 1.27)) hide)
     )
     (pin "1")
   )
-  (symbol (lib_id "power:GND") (at 117.856 91.694 0) (mirror y) (unit 1)
+  (symbol (lib_id "power:GND") (at 108.966 93.726 0) (mirror y) (unit 1)
     (in_bom yes) (on_board yes) (fields_autoplaced)
-    (property "Reference" "#PWR014" (id 0) (at 117.856 98.044 0)
+    (property "Reference" "#PWR014" (id 0) (at 108.966 100.076 0)
       (effects (font (size 1.27 1.27)) hide)
     )
-    (property "Value" "GND" (id 1) (at 117.856 96.1374 0))
-    (property "Footprint" "" (id 2) (at 117.856 91.694 0)
+    (property "Value" "GND" (id 1) (at 108.966 98.1694 0))
+    (property "Footprint" "" (id 2) (at 108.966 93.726 0)
       (effects (font (size 1.27 1.27)) hide)
     )
-    (property "Datasheet" "" (id 3) (at 117.856 91.694 0)
+    (property "Datasheet" "" (id 3) (at 108.966 93.726 0)
       (effects (font (size 1.27 1.27)) hide)
     )

Commit message: routing finished
Parts:
- removed U2: TLV76733DRVx, Package_TO_SOT_SMD:SOT-23-5_HandSoldering, symbol Regulator_Linear:TLV76733DRVx
- added U2: BD733L5FP-CE2, BD733L5FP:BD750L5FPCE2, symbol BD733L5FP:BD733L5FP-CE2
Connections:
- net +12V: now also U2.1 (VCC)
- net +3V3: now also U2.3 (VOUT)
- net GND: now also U2.4 (GND)
Other:
- moved on the sheet: C1

Commit message: Improve style
Other:
- note added: "Inverted because this is an XT30 actually"
- note removed: "Inverted because this and XT30 actually"
Changed lines of the file:
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@@
     (effects (font (size 2.5 2.5) (thickness 0.5) bold) (justify left bottom))
   )
-  (text "Inverted because this and XT30 actually" (at 83.82 102.87 0)
+  (text "Inverted because this is an XT30 actually" (at 83.82 102.87 0)
     (effects (font (size 1.27 1.27)) (justify left bottom))
   )
